Commit message: feat: Add MoveIt2 configuration for the rm75 robot with gripper and cameras, including new URDFs, SRDF, and launch files. TODO:fix launch robot_moveit_config bug

File: src/Two-finger Electric Gripper.urdf/urdf/EG2-4C2.urdf (robot description, URDF)
Before this commit: robot EG2-4C2, 7 links, 6 joints
Links:
- removed link 4C2_Link1
- removed link 4C2_Link2
- removed link 4C2_Link3
- removed link 4C2_Link4
- removed link 4C2_Link5
- removed link 4C2_Link6
- removed link 4C2_baselink
- added link eg2_4c2_baselink, mass 0.072633; collision mesh filename=package://eg2_4c2_description/meshes/4C2_baselink.STL; visual mesh filename=package://eg2_4c2_description/meshes/4C2_baselink.STL
- added link eg2_4c2_link1, mass 0.0024292; collision mesh filename=package://eg2_4c2_description/meshes/4C2_Link1.STL; visual mesh filename=package://eg2_4c2_description/meshes/4C2_Link1.STL
- added link eg2_4c2_link2, mass 0.0038971; collision mesh filename=package://eg2_4c2_description/meshes/4C2_Link2.STL; visual mesh filename=package://eg2_4c2_description/meshes/4C2_Link2.STL
- added link eg2_4c2_link3, mass 0.0038971; collision mesh filename=package://eg2_4c2_description/meshes/4C2_Link3.STL; visual mesh filename=package://eg2_4c2_description/meshes/4C2_Link3.STL
- added link eg2_4c2_link4, mass 0.0024292; collision mesh filename=package://eg2_4c2_description/meshes/4C2_Link4.STL; visual mesh filename=package://eg2_4c2_description/meshes/4C2_Link4.STL
- added link eg2_4c2_link5, mass 0.0045068; collision mesh filename=package://eg2_4c2_description/meshes/4C2_Link5.STL; visual mesh filename=package://eg2_4c2_description/meshes/4C2_Link5.STL
- added link eg2_4c2_link6, mass 0.0045068; collision mesh filename=package://eg2_4c2_description/meshes/4C2_Link6.STL; visual mesh filename=package://eg2_4c2_description/meshes/4C2_Link6.STL
Joints:
- removed joint 4C2_Joint1
- removed joint 4C2_Joint2
- removed joint 4C2_Joint3
- removed joint 4C2_Joint4
- removed joint 4C2_Joint5
- removed joint 4C2_Joint6
- added joint eg2_4c2_joint1: type revolute, parent eg2_4c2_baselink, child eg2_4c2_link1, origin xyz=-0.04 -0.009 0.079 rpy=0 0 0, axis 0 -1 0, limit lower=0 upper=0.82 effort=1 velocity=1
- added joint eg2_4c2_joint2: type revolute, parent eg2_4c2_baselink, child eg2_4c2_link2, origin xyz=-0.03 -0.009 0.081 rpy=0 0 0, axis 0 -1 0, limit lower=0 upper=0.82 effort=1 velocity=1, mimic joint=eg2_4c2_joint1
- added joint eg2_4c2_joint3: type revolute, parent eg2_4c2_baselink, child eg2_4c2_link3, origin xyz=0.03 -0.009 0.081 rpy=0 0 0, axis 0 -1 0, limit lower=-0.82 upper=0 effort=1 velocity=1, mimic joint=eg2_4c2_joint1 multiplier=-1 offset=0
- added joint eg2_4c2_joint4: type revolute, parent eg2_4c2_baselink, child eg2_4c2_link4, origin xyz=0.04 -0.009 0.079 rpy=0 0 0, axis 0 -1 0, limit lower=-0.82 upper=0 effort=1 velocity=1, mimic joint=eg2_4c2_joint1 multiplier=-1 offset=0
- added joint eg2_4c2_joint5: type revolute, parent eg2_4c2_link1, child eg2_4c2_link5, origin xyz=0.0223 0.003 0.035591 rpy=0 0 0, axis 0 1 0, limit lower=0 upper=0.82 effort=1 velocity=1, mimic joint=eg2_4c2_joint1
- added joint eg2_4c2_joint6: type revolute, parent eg2_4c2_link4, child eg2_4c2_link6, origin xyz=-0.0223 0.003 0.035591 rpy=0 0 0, axis 0 -1 0, limit lower=0 upper=0.82 effort=1 velocity=1, mimic joint=eg2_4c2_joint1
