Commit message: feat: Configure Gazebo simulation with fixed robot base, updated model paths, and automatic controller spawning.

File: src/robot_gazebo_sim/urdf/robot_system.urdf.xacro (robot description, xacro)
@@ -11,4 +11,11 @@
     <color rgba="0.75 0.75 0.75 1"/>
   </material>
+  <xacro:property name="rm75_mesh_dir" value="$(find rm_75_6f_description)/meshes"/>
+  <xacro:property name="gripper_mesh_dir" value="$(find robot_gazebo_sim)/meshes/gripper"/>
+  <!-- Fixed base to world for stable simulation -->
+  <link name="world"/>
+  <gazebo reference="world">
+    <static>true</static>
+  </gazebo>
   <!-- ==================== Base Link ==================== -->
   <link name="base_link">
@@ -21,15 +28,20 @@
       <origin xyz="0 0 0" rpy="0 0 0"/>
       <geometry>
-        <mesh filename="package://rm_75_6f_description/meshes/base_link.STL"/>
-      </geometry>
-      <material name="white"/>
-    </visual>
-    <collision>
-      <origin xyz="0 0 0" rpy="0 0 0"/>
-      <geometry>
-        <mesh filename="package://rm_75_6f_description/meshes/base_link.STL"/>
-      </geometry>
-    </collision>
-  </link>
+        <mesh filename="file://${rm75_mesh_dir}/base_link.STL"/>
+      </geometry>
+      <material name="white"/>
+    </visual>
+    <collision>
+      <origin xyz="0 0 0" rpy="0 0 0"/>
+      <geometry>
+        <mesh filename="file://${rm75_mesh_dir}/base_link.STL"/>
+      </geometry>
+    </collision>
+  </link>
+  <joint name="world_joint" type="fixed">
+    <origin xyz="0 0 0" rpy="0 0 0"/>
+    <parent link="world"/>
+    <child link="base_link"/>
+  </joint>
   <!-- RM-75-6F Robot Arm -->
   <!-- Link1 -->
@@ -43,12 +55,12 @@
       <origin xyz="0 0 0" rpy="0 0 0"/>
       <geometry>
-        <mesh filename="package://rm_75_6f_description/meshes/Link1.STL"/>
-      </geometry>
-      <material name="white"/>
-    </visual>
-    <collision>
-      <origin xyz="0 0 0" rpy="0 0 0"/>
-      <geometry>
-        <mesh filename="package://rm_75_6f_description/meshes/Link1.STL"/>
+        <mesh filename="file://${rm75_mesh_dir}/Link1.STL"/>
+      </geometry>
+      <material name="white"/>
+    </visual>
+    <collision>
+      <origin xyz="0 0 0" rpy="0 0 0"/>
+      <geometry>
+        <mesh filename="file://${rm75_mesh_dir}/Link1.STL"/>
       </geometry>
     </collision>
@@ -71,12 +83,12 @@
       <origin xyz="0 0 0" rpy="0 0 0"/>
       <geometry>
-        <mesh filename="package://rm_75_6f_description/meshes/Link2.STL"/>
-      </geometry>
-      <material name="white"/>
-    </visual>
-    <collision>
-      <origin xyz="0 0 0" rpy="0 0 0"/>
-      <geometry>
-        <mesh filename="package://rm_75_6f_description/meshes/Link2.STL"/>
+        <mesh filename="file://${rm75_mesh_dir}/Link2.STL"/>
+      </geometry>
+      <material name="white"/>
+    </visual>
+    <collision>
+      <origin xyz="0 0 0" rpy="0 0 0"/>
+      <geometry>
+        <mesh filename="file://${rm75_mesh_dir}/Link2.STL"/>
       </geometry>
     </collision>
@@ -99,12 +111,12 @@
       <origin xyz="0 0 0" rpy="0 0 0"/>
       <geometry>
-        <mesh filename="package://rm_75_6f_description/meshes/Link3.STL"/>
-      </geometry>
-      <material name="white"/>
-    </visual>
-    <collision>
-      <origin xyz="0 0 0" rpy="0 0 0"/>
-      <geometry>
-        <mesh filename="package://rm_75_6f_description/meshes/Link3.STL"/>
+        <mesh filename="file://${rm75_mesh_dir}/Link3.STL"/>
+      </geometry>
+      <material name="white"/>
+    </visual>
+    <collision>
+      <origin xyz="0 0 0" rpy="0 0 0"/>
+      <geometry>
+        <mesh filename="file://${rm75_mesh_dir}/Link3.STL"/>
       </geometry>
     </collision>
@@ -127,12 +139,12 @@
       <origin xyz="0 0 0" rpy="0 0 0"/>
       <geometry>
-        <mesh filename="package://rm_75_6f_description/meshes/Link4.STL"/>
-      </geometry>
-      <material name="white"/>
-    </visual>
-    <collision>
-      <origin xyz="0 0 0" rpy="0 0 0"/>
-      <geometry>
-        <mesh filename="package://rm_75_6f_description/meshes/Link4.STL"/>
+        <mesh filename="file://${rm75_mesh_dir}/Link4.STL"/>
+      </geometry>
+      <material name="white"/>
+    </visual>
+    <collision>
+      <origin xyz="0 0 0" rpy="0 0 0"/>
+      <geometry>
+        <mesh filename="file://${rm75_mesh_dir}/Link4.STL"/>
       </geometry>
     </collision>
@@ -155,12 +167,12 @@
       <origin xyz="0 0 0" rpy="0 0 0"/>
       <geometry>
-        <mesh filename="package://rm_75_6f_description/meshes/Link5.STL"/>
-      </geometry>
-      <material name="white"/>
-    </visual>
-    <collision>
-      <origin xyz="0 0 0" rpy="0 0 0"/>
-      <geometry>
-        <mesh filename="package://rm_75_6f_description/meshes/Link5.STL"/>
+        <mesh filename="file://${rm75_mesh_dir}/Link5.STL"/>
+      </geometry>
+      <material name="white"/>
+    </visual>
+    <collision>
+      <origin xyz="0 0 0" rpy="0 0 0"/>
+      <geometry>
+        <mesh filename="file://${rm75_mesh_dir}/Link5.STL"/>
       </geometry>
     </collision>
@@ -183,12 +195,12 @@
       <origin xyz="0 0 0" rpy="0 0 0"/>
       <geometry>
-        <mesh filename="package://rm_75_6f_description/meshes/Link6.STL"/>
-      </geometry>
-      <material name="white"/>
-    </visual>
-    <collision>
-      <origin xyz="0 0 0" rpy="0 0 0"/>
-      <geometry>
-        <mesh filename="package://rm_75_6f_description/meshes/Link6.STL"/>
+        <mesh filename="file://${rm75_mesh_dir}/Link6.STL"/>
+      </geometry>
+      <material name="white"/>
+    </visual>
+    <collision>
+      <origin xyz="0 0 0" rpy="0 0 0"/>
+      <geometry>
+        <mesh filename="file://${rm75_mesh_dir}/Link6.STL"/>
       </geometry>
     </collision>
@@ -211,12 +223,12 @@
       <origin xyz="0 0 0" rpy="0 0 0"/>
       <geometry>
-        <mesh filename="package://rm_75_6f_description/meshes/Link7.STL"/>
-      </geometry>
-      <material name="white"/>
-    </visual>
-    <collision>
-      <origin xyz="0 0 0" rpy="0 0 0"/>
-      <geometry>
-        <mesh filename="package://rm_75_6f_description/meshes/Link7.STL"/>
+        <mesh filename="file://${rm75_mesh_dir}/Link7.STL"/>
+      </geometry>
+      <material name="white"/>
+    </visual>
+    <collision>
+      <origin xyz="0 0 0" rpy="0 0 0"/>
+      <geometry>
+        <mesh filename="file://${rm75_mesh_dir}/Link7.STL"/>
       </geometry>
     </collision>
@@ -240,5 +252,5 @@
       <origin xyz="0 0 0" rpy="0 0 0"/>
       <geometry>
-        <mesh filename="package://robot_gazebo_sim/meshes/gripper/4C2_baselink.STL"/>
+        <mesh filename="file://${gripper_mesh_dir}/4C2_baselink.STL"/>
       </geometry>
       <material name="grey"/>
@@ -247,5 +259,5 @@
       <origin xyz="0 0 0" rpy="0 0 0"/>
       <geometry>
-        <mesh filename="package://robot_gazebo_sim/meshes/gripper/4C2_baselink.STL"/>
+        <mesh filename="file://${gripper_mesh_dir}/4C2_baselink.STL"/>
       </geometry>
     </collision>
@@ -267,5 +279,5 @@
       <origin xyz="0 0 0" rpy="0 0 0"/>
       <geometry>
-        <mesh filename="package://robot_gazebo_sim/meshes/gripper/4C2_Link1.STL"/>
+        <mesh filename="file://${gripper_mesh_dir}/4C2_Link1.STL"/>
       </geometry>
       <material name="grey"/>
@@ -274,5 +286,5 @@
       <origin xyz="0 0 0" rpy="0 0 0"/>
       <geometry>
-        <mesh filename="package://robot_gazebo_sim/meshes/gripper/4C2_Link1.STL"/>
+        <mesh filename="file://${gripper_mesh_dir}/4C2_Link1.STL"/>
       </geometry>
     </collision>
@@ -294,5 +306,5 @@
       <origin xyz="0 0 0" rpy="0 0 0"/>
       <geometry>
-        <mesh filename="package://robot_gazebo_sim/meshes/gripper/4C2_Link5.STL"/>
+        <mesh filename="file://${gripper_mesh_dir}/4C2_Link5.STL"/>
       </geometry>
       <material name="grey"/>
@@ -301,5 +313,5 @@
       <origin xyz="0 0 0" rpy="0 0 0"/>
       <geometry>
-        <mesh filename="package://robot_gazebo_sim/meshes/gripper/4C2_Link5.STL"/>
+        <mesh filename="file://${gripper_mesh_dir}/4C2_Link5.STL"/>
       </geometry>
     </collision>
@@ -322,5 +334,5 @@
       <origin xyz="0 0 0" rpy="0 0 0"/>
       <geometry>
-        <mesh filename="package://robot_gazebo_sim/meshes/gripper/4C2_Link4.STL"/>
+        <mesh filename="file://${gripper_mesh_dir}/4C2_Link4.STL"/>
       </geometry>
       <material name="grey"/>
@@ -329,5 +341,5 @@
       <origin xyz="0 0 0" rpy="0 0 0"/>
       <geometry>
-        <mesh filename="package://robot_gazebo_sim/meshes/gripper/4C2_Link4.STL"/>
+        <mesh filename="file://${gripper_mesh_dir}/4C2_Link4.STL"/>
       </geometry>
     </collision>
@@ -350,5 +362,5 @@
       <origin xyz="0 0 0" rpy="0 0 0"/>
       <geometry>
-        <mesh filename="package://robot_gazebo_sim/meshes/gripper/4C2_Link6.STL"/>
+        <mesh filename="file://${gripper_mesh_dir}/4C2_Link6.STL"/>
       </geometry>
       <material name="grey"/>
@@ -357,5 +369,5 @@
       <origin xyz="0 0 0" rpy="0 0 0"/>
       <geometry>
-        <mesh filename="package://robot_gazebo_sim/meshes/gripper/4C2_Link6.STL"/>
+        <mesh filename="file://${gripper_mesh_dir}/4C2_Link6.STL"/>
       </geometry>
     </collision>

Commit message: feat: fix launch robot_moveit_config bug 但是gazebo掉落抖动问题依旧没解决，导致moveit的execute也有问题

File: src/robot_gazebo_sim/urdf/robot_system.urdf.xacro (robot description, xacro)
@@ -1,4 +1,5 @@
 <?xml version="1.0"?>
 <robot xmlns:xacro="http://www.ros.org/wiki/xacro" name="rm75_gripper_cameras">
+  <xacro:arg name="use_gazebo_control" default="true"/>
   <!-- Include component xacro files -->
   <xacro:include filename="$(find robot_gazebo_sim)/urdf/realsense_d405.urdf.xacro"/>
@@ -390,78 +391,80 @@
   </xacro:realsense_d435>
   <!-- ==================== ROS2 Control ==================== -->
-  <ros2_control name="GazeboSystem" type="system">
-    <hardware>
-      <plugin>gazebo_ros2_control/GazeboSystem</plugin>
-    </hardware>
-    <joint name="joint1">
-      <command_interface name="position">
-        <param name="min">-3.107</param>
-        <param name="max">3.107</param>
-      </command_interface>
-      <state_interface name="position"/>
-      <state_interface name="velocity"/>
-    </joint>
-    <joint name="joint2">
-      <command_interface name="position">
-        <param name="min">-2.269</param>
-        <param name="max">2.269</param>
-      </command_interface>
-      <state_interface name="position"/>
-      <state_interface name="velocity"/>
-    </joint>
-    <joint name="joint3">
-      <command_interface name="position">
-        <param name="min">-3.107</param>
-        <param name="max">3.107</param>
-      </command_interface>
-      <state_interface name="position"/>
-      <state_interface name="velocity"/>
-    </joint>
-    <joint name="joint4">
-      <command_interface name="position">
-        <param name="min">-2.356</param>
-        <param name="max">2.356</param>
-      </command_interface>
-      <state_interface name="position"/>
-      <state_interface name="velocity"/>
-    </joint>
-    <joint name="joint5">
-      <command_interface name="position">
-        <param name="min">-3.107</param>
-        <param name="max">3.107</param>
-      </command_interface>
-      <state_interface name="position"/>
-      <state_interface name="velocity"/>
-    </joint>
-    <joint name="joint6">
-      <command_interface name="position">
-        <param name="min">-2.234</param>
-        <param name="max">2.234</param>
-      </command_interface>
-      <state_interface name="position"/>
-      <state_interface name="velocity"/>
-    </joint>
-    <joint name="joint7">
-      <command_interface name="position">
-        <param name="min">-6.283</param>
-        <param name="max">6.283</param>
-      </command_interface>
-      <state_interface name="position"/>
-      <state_interface name="velocity"/>
-    </joint>
-    <joint name="gripper_finger1_joint">
-      <command_interface name="position"/>
-      <state_interface name="position"/>
-      <state_interface name="velocity"/>
-    </joint>
-  </ros2_control>
-  <!-- ==================== Gazebo Properties ==================== -->
-  <gazebo>
-    <plugin filename="libgazebo_ros2_control.so" name="gazebo_ros2_control">
-      <robot_param>robot_description</robot_param>
-      <robot_param_node>robot_state_publisher</robot_param_node>
-      <parameters>$(find robot_gazebo_sim)/config/controllers.yaml</parameters>
-    </plugin>
-  </gazebo>
+  <xacro:if value="${xacro.arg('use_gazebo_control')}">
+    <ros2_control name="GazeboSystem" type="system">
+      <hardware>
+        <plugin>gazebo_ros2_control/GazeboSystem</plugin>
+      </hardware>
+      <joint name="joint1">
+        <command_interface name="position">
+          <param name="min">-3.107</param>
+          <param name="max">3.107</param>
+        </command_interface>
+        <state_interface name="position"/>
+        <state_interface name="velocity"/>
+      </joint>
+      <joint name="joint2">
+        <command_interface name="position">
+          <param name="min">-2.269</param>
+          <param name="max">2.269</param>
+        </command_interface>
+        <state_interface name="position"/>
+        <state_interface name="velocity"/>
+      </joint>
+      <joint name="joint3">
+        <command_interface name="position">
+          <param name="min">-3.107</param>
+          <param name="max">3.107</param>
+        </command_interface>
+        <state_interface name="position"/>
+        <state_interface name="velocity"/>
+      </joint>
+      <joint name="joint4">
+        <command_interface name="position">
+          <param name="min">-2.356</param>
+          <param name="max">2.356</param>
+        </command_interface>
+        <state_interface name="position"/>
+        <state_interface name="velocity"/>
+      </joint>
+      <joint name="joint5">
+        <command_interface name="position">
+          <param name="min">-3.107</param>
+          <param name="max">3.107</param>
+        </command_interface>
+        <state_interface name="position"/>
+        <state_interface name="velocity"/>
+      </joint>
+      <joint name="joint6">
+        <command_interface name="position">
+          <param name="min">-2.234</param>
+          <param name="max">2.234</param>
+        </command_interface>
+        <state_interface name="position"/>
+        <state_interface name="velocity"/>
+      </joint>
+      <joint name="joint7">
+        <command_interface name="position">
+          <param name="min">-6.283</param>
+          <param name="max">6.283</param>
+        </command_interface>
+        <state_interface name="position"/>
+        <state_interface name="velocity"/>
+      </joint>
+      <joint name="gripper_finger1_joint">
+        <command_interface name="position"/>
+        <state_interface name="position"/>
+        <state_interface name="velocity"/>
+      </joint>
+    </ros2_control>
+    <!-- ==================== Gazebo Properties ==================== -->
+    <gazebo>
+      <plugin filename="libgazebo_ros2_control.so" name="gazebo_ros2_control">
+        <robot_param>robot_description</robot_param>
+        <robot_param_node>robot_state_publisher</robot_param_node>
+        <parameters>$(find robot_gazebo_sim)/config/controllers.yaml</parameters>
+      </plugin>
+    </gazebo>
+  </xacro:if>
   <!-- Arm joint Gazebo properties -->
   <gazebo reference="base_link">

File: src/robot_moveit_config/config/rm75_gripper_cameras.urdf.xacro (robot description, xacro)
@@ -2,8 +2,15 @@
 <robot xmlns:xacro="http://www.ros.org/wiki/xacro" name="rm75_gripper_cameras">
     <xacro:arg name="initial_positions_file" default="initial_positions.yaml" />
+    <xacro:arg name="use_fake_hardware" default="true" />
+    <xacro:arg name="use_gazebo_control" default="false" />
     <!-- Import rm75_gripper_cameras urdf file -->
+    <!-- Pass use_gazebo_control to base URDF to control hardware plugin loading -->
     <xacro:include filename="$(find robot_gazebo_sim)/urdf/robot_system.urdf.xacro" />
-    <!-- Import control_xacro -->
-    <xacro:include filename="rm75_gripper_cameras.ros2_control.xacro" />
-    <xacro:rm75_gripper_cameras_ros2_control name="FakeSystem" initial_positions_file="$(arg initial_positions_file)"/>
+    <!-- Only include fake hardware ros2_control when needed (for MoveIt2 demo without Gazebo) -->
+    <xacro:if value="$(arg use_fake_hardware)">
+        <xacro:include filename="rm75_gripper_cameras.ros2_control.xacro" />
+        <xacro:rm75_gripper_cameras_ros2_control
+            name="FakeSystem"
+            initial_positions_file="$(arg initial_positions_file)"/>
+    </xacro:if>
 </robot>
