Commit message: 问题:gazebo加载的机械臂link和joint都在原点

File: src/robot_gazebo_sim/urdf/robot_system.urdf.xacro (robot description, xacro)
@@ -15,7 +15,4 @@
   <!-- Fixed base to world for stable simulation -->
   <link name="world"/>
-  <gazebo reference="world">
-    <static>true</static>
-  </gazebo>
   <!-- ==================== Base Link ==================== -->
   <link name="base_link">
@@ -453,49 +450,62 @@
   <gazebo reference="base_link">
     <material>Gazebo/White</material>
+    <gravity>false</gravity>
   </gazebo>
   <gazebo reference="Link1">
     <material>Gazebo/White</material>
+    <gravity>false</gravity>
   </gazebo>
   <gazebo reference="Link2">
     <material>Gazebo/White</material>
+    <gravity>false</gravity>
   </gazebo>
   <gazebo reference="Link3">
     <material>Gazebo/White</material>
+    <gravity>false</gravity>
   </gazebo>
   <gazebo reference="Link4">
     <material>Gazebo/White</material>
+    <gravity>false</gravity>
   </gazebo>
   <gazebo reference="Link5">
     <material>Gazebo/White</material>
+    <gravity>false</gravity>
   </gazebo>
   <gazebo reference="Link6">
     <material>Gazebo/White</material>
+    <gravity>false</gravity>
   </gazebo>
   <gazebo reference="Link7">
     <material>Gazebo/White</material>
+    <gravity>false</gravity>
   </gazebo>
   <!-- Gripper Gazebo properties -->
   <gazebo reference="gripper_base_link">
     <material>Gazebo/Grey</material>
+    <gravity>false</gravity>
   </gazebo>
   <gazebo reference="gripper_finger1_link">
     <material>Gazebo/Grey</material>
-    <kp>1000000.0</kp>
-    <kd>100.0</kd>
-    <mu1>1.0</mu1>
-    <mu2>1.0</mu2>
+    <gravity>false</gravity>
   </gazebo>
   <gazebo reference="gripper_finger1_link2">
     <material>Gazebo/Grey</material>
+    <gravity>false</gravity>
+  </gazebo>
+  <gazebo reference="gripper_finger1_tip_link">
+    <material>Gazebo/Grey</material>
+    <gravity>false</gravity>
   </gazebo>
   <gazebo reference="gripper_finger2_link">
     <material>Gazebo/Grey</material>
-    <kp>1000000.0</kp>
-    <kd>100.0</kd>
-    <mu1>1.0</mu1>
-    <mu2>1.0</mu2>
+    <gravity>false</gravity>
   </gazebo>
   <gazebo reference="gripper_finger2_link3">
     <material>Gazebo/Grey</material>
+    <gravity>false</gravity>
+  </gazebo>
+  <gazebo reference="gripper_finger2_tip_link">
+    <material>Gazebo/Grey</material>
+    <gravity>false</gravity>
   </gazebo>
 </robot>

File: src/robot_moveit_config/config/rm75_gripper_cameras.gazebo_ros2_control.xacro (robot description, xacro)
@@ -1,5 +1,4 @@
 <?xml version="1.0"?>
 <robot xmlns:xacro="http://www.ros.org/wiki/xacro">
-    <!-- Gazebo System ros2_control macro -->
     <xacro:macro name="rm75_gripper_cameras_gazebo_ros2_control" params="controllers_file">
         <ros2_control name="GazeboSystem" type="system">
@@ -7,107 +6,68 @@
                 <plugin>gazebo_ros2_control/GazeboSystem</plugin>
             </hardware>
+            <!-- Arm Joints -->
             <joint name="joint1">
-                <command_interface name="position">
-                    <param name="min">-3.107</param>
-                    <param name="max">3.107</param>
-                </command_interface>
-                <state_interface name="position"/>
+                <command_interface name="position"/>
+                <state_interface name="position">
+                    <param name="initial_value">0</param>
+                </state_interface>
                 <state_interface name="velocity"/>
             </joint>
             <joint name="joint2">
-                <command_interface name="position">
-                    <param name="min">-2.269</param>
-                    <param name="max">2.269</param>
-                </command_interface>
-                <state_interface name="position"/>
+                <command_interface name="position"/>
+                <state_interface name="position">
+                    <param name="initial_value">0</param>
+                </state_interface>
                 <state_interface name="velocity"/>
             </joint>
             <joint name="joint3">
-                <command_interface name="position">
-                    <param name="min">-3.107</param>
-                    <param name="max">3.107</param>
-                </command_interface>
-                <state_interface name="position"/>
+                <command_interface name="position"/>
+                <state_interface name="position">
+                    <param name="initial_value">0</param>
+                </state_interface>
                 <state_interface name="velocity"/>
             </joint>
             <joint name="joint4">
-                <command_interface name="position">
-                    <param name="min">-2.356</param>
-                    <param name="max">2.356</param>
-                </command_interface>
-                <state_interface name="position"/>
+                <command_interface name="position"/>
+                <state_interface name="position">
+                    <param name="initial_value">0</param>
+                </state_interface>
                 <state_interface name="velocity"/>
             </joint>
             <joint name="joint5">
-                <command_interface name="position">
-                    <param name="min">-3.107</param>
-                    <param name="max">3.107</param>
-                </command_interface>
-                <state_interface name="position"/>
+                <command_interface name="position"/>
+                <state_interface name="position">
+                    <param name="initial_value">0</param>
+                </state_interface>
                 <state_interface name="velocity"/>
             </joint>
             <joint name="joint6">
-                <command_interface name="position">
-                    <param name="min">-2.234</param>
-                    <param name="max">2.234</param>
-                </command_interface>
-                <state_interface name="position"/>
+                <command_interface name="position"/>
+                <state_interface name="position">
+                    <param name="initial_value">0</param>
+                </state_interface>
                 <state_interface name="velocity"/>
             </joint>
             <joint name="joint7">
-                <command_interface name="position">
-                    <param name="min">-6.283</param>
-                    <param name="max">6.283</param>
-                </command_interface>
-                <state_interface name="position"/>
+                <command_interface name="position"/>
+                <state_interface name="position">
+                    <param name="initial_value">0</param>
+                </state_interface>
                 <state_interface name="velocity"/>
             </joint>
+            <!-- Gripper Joints -->
             <joint name="gripper_finger1_joint">
                 <command_interface name="position"/>
-                <state_interface name="position"/>
-                <state_interface name="velocity"/>
-            </joint>
-            <joint name="gripper_finger1_link2_joint">
-                <param name="mimic">gripper_finger1_joint</param>
-                <param name="multiplier">1</param>
-                <command_interface name="position"/>
-                <state_interface name="position"/>
-                <state_interface name="velocity"/>
-            </joint>
-            <joint name="gripper_finger2_joint">
-                <param name="mimic">gripper_finger1_joint</param>
-                <param name="multiplier">-1</param>
-                <command_interface name="position"/>
-                <state_interface name="position"/>
-                <state_interface name="velocity"/>
-            </joint>
-            <joint name="gripper_finger2_link3_joint">
-                <param name="mimic">gripper_finger1_joint</param>
-                <param name="multiplier">-1</param>
-                <command_interface name="position"/>
-                <state_interface name="position"/>
-                <state_interface name="velocity"/>
-            </joint>
-            <joint name="gripper_finger1_tip_joint">
-                <param name="mimic">gripper_finger1_joint</param>
-                <param name="multiplier">1</param>
-                <command_interface name="position"/>
-                <state_interface name="position"/>
-                <state_interface name="velocity"/>
-            </joint>
-            <joint name="gripper_finger2_tip_joint">
-                <param name="mimic">gripper_finger1_joint</param>
-                <param name="multiplier">1</param>
-                <command_interface name="position"/>
-                <state_interface name="position"/>
+                <state_interface name="position">
+                    <param name="initial_value">0</param>
+                </state_interface>
                 <state_interface name="velocity"/>
             </joint>
         </ros2_control>
-        <!-- Gazebo ros2_control plugin -->
         <gazebo>
             <plugin filename="libgazebo_ros2_control.so" name="gazebo_ros2_control">
+                <parameters>${controllers_file}</parameters>
                 <robot_param>robot_description</robot_param>
                 <robot_param_node>robot_state_publisher</robot_param_node>
-                <parameters>${controllers_file}</parameters>
             </plugin>
         </gazebo>

File: src/robot_moveit_config/config/rm75_gripper_cameras.ros2_control.xacro (robot description, xacro)
@@ -2,5 +2,5 @@
 <robot xmlns:xacro="http://www.ros.org/wiki/xacro">
     <xacro:macro name="rm75_gripper_cameras_ros2_control" params="name initial_positions_file">
-        <xacro:property name="initial_positions" value="${load_yaml(initial_positions_file)['initial_positions']}"/>
+        <xacro:property name="initial_positions" value="${xacro.load_yaml(initial_positions_file)['initial_positions']}"/>
         <ros2_control name="${name}" type="system">
             <hardware>
@@ -64,49 +64,4 @@
                 <state_interface name="velocity"/>
             </joint>
-            <joint name="gripper_finger1_link2_joint">
-                <param name="mimic">gripper_finger1_joint</param>
-                <param name="multiplier">1</param>
-                <command_interface name="position"/>
-                <state_interface name="position">
-                  <param name="initial_value">${initial_positions['gripper_finger1_link2_joint']}</param>
-                </state_interface>
-                <state_interface name="velocity"/>
-            </joint>
-            <joint name="gripper_finger2_joint">
-                <param name="mimic">gripper_finger1_joint</param>
-                <param name="multiplier">-1</param>
-                <command_interface name="position"/>
-                <state_interface name="position">
-                  <param name="initial_value">${initial_positions['gripper_finger2_joint']}</param>
-                </state_interface>
-                <state_interface name="velocity"/>
-            </joint>
-            <joint name="gripper_finger2_link3_joint">
-                <param name="mimic">gripper_finger1_joint</param>
-                <param name="multiplier">-1</param>
-                <command_interface name="position"/>
-                <state_interface name="position">
-                  <param name="initial_value">${initial_positions['gripper_finger2_link3_joint']}</param>
-                </state_interface>
-                <state_interface name="velocity"/>
-            </joint>
-            <joint name="gripper_finger1_tip_joint">
-                <param name="mimic">gripper_finger1_joint</param>
-                <param name="multiplier">1</param>
-                <command_interface name="position"/>
-                <state_interface name="position">
-                  <param name="initial_value">${initial_positions['gripper_finger1_tip_joint']}</param>
-                </state_interface>
-                <state_interface name="velocity"/>
-            </joint>
-            <joint name="gripper_finger2_tip_joint">
-                <param name="mimic">gripper_finger1_joint</param>
-                <param name="multiplier">1</param>
-                <command_interface name="position"/>
-                <state_interface name="position">
-                  <param name="initial_value">${initial_positions['gripper_finger2_tip_joint']}</param>
-                </state_interface>
-                <state_interface name="velocity"/>
-            </joint>
         </ros2_control>
     </xacro:macro>

File: src/robot_moveit_config/config/rm75_gripper_cameras.urdf.xacro (robot description, xacro)
@@ -5,5 +5,5 @@
     <xacro:arg name="use_gazebo" default="false" />
     <xacro:arg name="gazebo_controllers_file" default="" />
-    <!-- Import robot URDF from description package -->
+    <!-- Import rm75_gripper_cameras urdf file -->
     <xacro:include filename="$(find robot_gazebo_sim)/urdf/robot_system.urdf.xacro" />
     <!-- ros2_control for MoveIt2 fake hardware demo (mock hardware) -->

Commit message: feat: 修复gazebo加载机械臂有问题的bug TODO: 搭建环境

File: src/robot_gazebo_sim/urdf/robot_system.urdf.xacro (robot description, xacro)
@@ -348,5 +348,5 @@
     <child link="gripper_finger1_tip_link"/>
     <axis xyz="0 1 0"/>
-    <dynamics damping="1.0" friction="0.2"/>
+    <!-- <dynamics damping="1.0" friction="0.2"/> -->
     <limit lower="0" upper="0.82" effort="1" velocity="1"/>
     <mimic joint="gripper_finger1_joint"/>
@@ -434,7 +434,33 @@
     <child link="gripper_finger2_tip_link"/>
     <axis xyz="0 -1 0"/>
-    <dynamics damping="1.0" friction="0.2"/>
+    <!-- <dynamics damping="1.0" friction="0.2"/> -->
     <limit lower="0" upper="0.82" effort="1" velocity="1"/>
     <mimic joint="gripper_finger1_joint"/>
+  </joint>
+  <!-- https://github.com/ros-controls/gazebo_ros2_control/issues/173 -->
+  <link name="dummy_child1"/>
+  <link name="dummy_child2"/>
+  <link name="dummy_child3"/>
+  <link name="dummy_child4"/>
+  <link name="dummy_child5"/>
+  <joint name="gripper_finger1_link2_joint_mimic" type="fixed">
+      <parent link="gripper_base_link" />
+      <child link="dummy_child1" />
+  </joint>
+  <joint name="gripper_finger1_tip_joint_mimic" type="fixed">
+      <parent link="gripper_finger1_link" />
+      <child link="dummy_child2" />
+  </joint>
+  <joint name="gripper_finger2_joint_mimic" type="fixed">
+      <parent link="gripper_base_link" />
+      <child link="dummy_child3" />
+  </joint>
+  <joint name="gripper_finger2_link3_joint_mimic" type="fixed">
+      <parent link="gripper_base_link" />
+      <child link="dummy_child4" />
+  </joint>
+  <joint name="gripper_finger2_tip_joint_mimic" type="fixed">
+      <parent link="gripper_finger2_link" />
+      <child link="dummy_child5" />
   </joint>
   <!-- ==================== RealSense D405 (Eye-in-Hand) ==================== -->

File: src/robot_moveit_config/config/rm75_gripper_cameras.gazebo_ros2_control.xacro (robot description, xacro)
@@ -64,10 +64,43 @@
                 <state_interface name="velocity"/>
             </joint>
+            <joint name="gripper_finger1_link2_joint">
+                <param name="mimic">gripper_finger1_joint</param>
+                <param name="multiplier">1</param>
+                <command_interface name="position"/>
+                <state_interface name="position"/>
+                <state_interface name="velocity"/>
+            </joint>
+            <joint name="gripper_finger2_joint">
+                <param name="mimic">gripper_finger1_joint</param>
+                <param name="multiplier">-1</param>
+                <command_interface name="position"/>
+                <state_interface name="position"/>
+                <state_interface name="velocity"/>
+            </joint>
+            <joint name="gripper_finger2_link3_joint">
+                <param name="mimic">gripper_finger1_joint</param>
+                <param name="multiplier">-1</param>
+                <command_interface name="position"/>
+                <state_interface name="position"/>
+                <state_interface name="velocity"/>
+            </joint>
+            <joint name="gripper_finger1_tip_joint">
+                <param name="mimic">gripper_finger1_joint</param>
+                <param name="multiplier">1</param>
+                <command_interface name="position"/>
+                <state_interface name="position"/>
+                <state_interface name="velocity"/>
+            </joint>
+            <joint name="gripper_finger2_tip_joint">
+                <param name="mimic">gripper_finger1_joint</param>
+                <param name="multiplier">1</param>
+                <command_interface name="position"/>
+                <state_interface name="position"/>
+                <state_interface name="velocity"/>
+            </joint>
         </ros2_control>
         <gazebo>
             <plugin filename="libgazebo_ros2_control.so" name="gazebo_ros2_control">
                 <parameters>${controllers_file}</parameters>
-                <robot_param>robot_description</robot_param>
-                <robot_param_node>robot_state_publisher</robot_param_node>
             </plugin>
         </gazebo>

Commit message: feat: 新的gazebo环境，调整d405方向 TODO: gazebo中加上燕麦工件

File: src/robot_gazebo_sim/urdf/robot_system.urdf.xacro (robot description, xacro)
@@ -466,9 +466,9 @@
   <!-- ==================== RealSense D405 (Eye-in-Hand) ==================== -->
   <xacro:realsense_d405 name="d405" parent="gripper_base_link">
-    <origin xyz="0 0.04 0.04" rpy="0 ${pi/6} ${pi/2}"/>
+    <origin xyz="0 0.04 0.04" rpy="0 ${-pi/2} ${pi/2}"/>
   </xacro:realsense_d405>
   <!-- ==================== RealSense D435 (Eye-to-Hand) ==================== -->
   <xacro:realsense_d435 name="d435" parent="base_link">
-    <origin xyz="-0.4 0.8 0.45" rpy="0 0.6 ${-pi/2}"/>
+    <origin xyz="1.2 0 1" rpy="0 0.785398163 ${pi}"/>
   </xacro:realsense_d435>
   <!-- Note:ros2_control and Gazebo control plugins are defined in robot_moveit_config -->

Commit message: feat: 将world的obj改为stl，显示正常；调整相机位置，更靠近桌面

File: src/robot_gazebo_sim/urdf/robot_system.urdf.xacro (robot description, xacro)
@@ -470,5 +470,5 @@
   <!-- ==================== RealSense D435 (Eye-to-Hand) ==================== -->
   <xacro:realsense_d435 name="d435" parent="base_link">
-    <origin xyz="1.2 0 1" rpy="0 0.785398163 ${pi}"/>
+    <origin xyz="0.7 0 0.4" rpy="0 0.785398163 ${pi}"/>
   </xacro:realsense_d435>
   <!-- Note:ros2_control and Gazebo control plugins are defined in robot_moveit_config -->

Commit message: feat: 调整相机位置和关节速度/加速度限制以优化仿真性能

File: src/robot_gazebo_sim/urdf/robot_system.urdf.xacro (robot description, xacro)
@@ -506,5 +506,5 @@
   <!-- ==================== RealSense D435 (Eye-to-Hand) ==================== -->
   <xacro:realsense_d435 name="d435" parent="base_link">
-    <origin xyz="0.7 0 0.4" rpy="0 0.785398163 ${pi}"/>
+    <origin xyz="0.65 0 0.35" rpy="0 0.805398163 ${pi}"/>
   </xacro:realsense_d435>
   <!-- Note:ros2_control and Gazebo control plugins are defined in robot_moveit_config -->
